Commit message: added camera to the robot

File: R2/src/mecanumbot_description/urdf/mecanumbot.urdf.xacro (robot description, xacro)
@@ -210,4 +210,48 @@
     <material>Gazebo/Grey</material>
   </gazebo>
+  <joint name="camera_joint" type="fixed">
+    <parent link="base_link" />
+    <child link="camera_link" />
+    <origin xyz="-0.22 0 0.1" rpy="0 0 ${M_PI}" />
+  </joint>
+  <link name="camera_link">
+    <visual>
+      <geometry>
+        <box size="0.05 0.05 0.05" />
+      </geometry>
+      <material name="blue" />
+    </visual>
+    <inertial>
+      <mass value="0.1" />
+      <origin xyz="0 0 0" rpy="0 0 0" />
+      <inertia ixx="0.0001" ixy="0" ixz="0" iyy="0.0001" iyz="0" izz="0.0001" />
+    </inertial>
+  </link>
+  <gazebo reference="camera_link">
+    <sensor type="camera" name="camera">
+      <update_rate>30.0</update_rate>
+      <topic>/camera/image_raw</topic>
+      <camera name="head">
+        <horizontal_fov>1.3962634</horizontal_fov>
+        <image>
+          <width>800</width>
+          <height>600</height>
+          <format>R8G8B8</format>
+        </image>
+        <clip>
+          <near>0.02</near>
+          <far>300</far>
+        </clip>
+        <noise>
+          <type>gaussian</type>
+          <mean>0.0</mean>
+          <stddev>0.007</stddev>
+        </noise>
+      </camera>
+      <always_on>1</always_on>
+      <visualize>true</visualize>
+    </sensor>
+    <material>Gazebo/Blue</material>
+  </gazebo>
   <gazebo>
     <plugin filename="libgz_ros2_control-system.so" name="gz_ros2_control::GazeboSimROS2ControlPlugin">

Commit message: feat : maps robot mecanum joy stick

File: R2/src/mecanumbot_description/urdf/mecanumbot.urdf.xacro (robot description, xacro)
@@ -167,7 +167,7 @@
   <ros2_control name="mecanumbot" type="system">
     <hardware>
-      <plugin>gz_ros2_control/GazeboSimSystem</plugin>
+      <plugin>ign_ros2_control/IgnitionSystem</plugin>
     </hardware>
-    <joint name="fl_wheel_joint">
+    <joint name="FL_wheel_joint">
       <command_interface name="velocity" />
       <state_interface name="position" />
@@ -175,5 +175,5 @@
       <param name="motor_id">1</param>
     </joint>
-    <joint name="fr_wheel_joint">
+    <joint name="FR_wheel_joint">
       <command_interface name="velocity" />
       <state_interface name="position" />
@@ -181,5 +181,5 @@
       <param name="motor_id">2</param>
     </joint>
-    <joint name="rl_wheel_joint">
+    <joint name="RL_wheel_joint">
       <command_interface name="velocity" />
       <state_interface name="position" />
@@ -187,5 +187,5 @@
       <param name="motor_id">4</param>
     </joint>
-    <joint name="rr_wheel_joint">
+    <joint name="RR_wheel_joint">
       <command_interface name="velocity" />
       <state_interface name="position" />
@@ -195,21 +195,23 @@
   </ros2_control>
   <!-- Gazebo-specific configurations for wheels -->
-  <gazebo reference="fl_wheel_link">
-    <material>Gazebo/DarkGrey</material>
-  </gazebo>
-  <gazebo reference="fr_wheel_link">
-    <material>Gazebo/DarkGrey</material>
-  </gazebo>
-  <gazebo reference="rl_wheel_link">
-    <material>Gazebo/DarkGrey</material>
-  </gazebo>
-  <gazebo reference="rr_wheel_link">
+  <gazebo reference="FL_wheel_link">
+    <material>Gazebo/DarkGrey</material>
+  </gazebo>
+  <gazebo reference="FR_wheel_link">
+    <material>Gazebo/DarkGrey</material>
+  </gazebo>
+  <gazebo reference="RL_wheel_link">
+    <material>Gazebo/DarkGrey</material>
+  </gazebo>
+  <gazebo reference="RR_wheel_link">
     <material>Gazebo/DarkGrey</material>
   </gazebo>
   <gazebo reference="base_link">
     <material>Gazebo/Grey</material>
+    <gravity>true</gravity>
+    <kinematic>false</kinematic>
   </gazebo>
   <gazebo>
-    <plugin filename="libgz_ros2_control-system.so" name="gz_ros2_control::GazeboSimROS2ControlPlugin">
+    <plugin filename="libign_ros2_control-system.so" name="ign_ros2_control::IgnitionROS2ControlPlugin">
       <parameters>$(find mecanumbot_description)/config/robot_controller_config.yaml</parameters>
     </plugin>

Commit message: just in case (STILL DOESNT WORKS)

File: R2/src/mecanumbot_description/urdf/mecanumbot.urdf.xacro (robot description, xacro)
@@ -213,5 +213,5 @@
     <parent link="base_link" />
     <child link="camera_link" />
-    <origin xyz="-0.22 0 0.1" rpy="0 0 ${M_PI}" />
+    <origin xyz="0.12 0.0 0.1" rpy="0 0 0" />
   </joint>
   <link name="camera_link">

Commit message: fixed apriltag_distance_node and tag_follower_node. also readme complete

File: R2/src/mecanumbot_description/urdf/mecanumbot.urdf.xacro (robot description, xacro)
@@ -213,5 +213,5 @@
     <parent link="base_link" />
     <child link="camera_link" />
-    <origin xyz="0.12 0.0 0.1" rpy="0 0 0" />
+    <origin xyz="-0.12 0.0 0.1" rpy="0 0 3.14159" />
   </joint>
   <link name="camera_link">
